File: Attiny2x4x8x Programmers.kicad_sch (KiCad schematic)
At the start: 9 parts, among them J1 Conn_01x15_Pin, J2 Conn_01x15_Pin, J3 ICSP, U1 ATtiny84-20P, U2 ATtiny85V-10P

Commit message: V2
Parts:
- added SW1: OS102011MS2QN1, OS102011MS2QN1:SPDT_OS102011_CNK, symbol OS102011MS2QN1:OS102011MS2QN1
Connections:
- net RST: now also SW1.1; no longer C1.1
- new net: C1.1, SW1.2, SW1.3
Other:
- moved on the sheet: A1, C1, D1, J1, J2, J3, R1, U1, U2
